File: schematics/propeller-clock-schematic.sch (KiCad schematic (older format))
At the start: 0 parts

Commit message: saved project
Parts:
- added J?: TEST, symbol TEST
Changed lines of the file:
@@
-EESchema Schematic File Version 2  date Monday, 2013 January 07 23:56:14
+EESchema Schematic File Version 2  date Tuesday, 2013 January 08 00:16:28
+LIBS:propeller-clock-components
 EELAYER 27 0
 EELAYER END
@@
 Comment4 ""
 $EndDescr
+$Comp
+L TEST J?
+U 1 1 50EB5748
+P 3950 1800
+F 0 "J?" H 3950 1800 60  0000 C CNN
+F 1 "TEST" H 3950 1800 60  0000 C CNN
+	1    3950 1800
+	1    0    0    -1
+$EndComp
 $EndSCHEMATC
